File: 2. Projects/2. PCB Implementation/PCB design/vending_machine_pcb/Coin_Buttons.kicad_sch (KiCad schematic)
At the start: 6 parts, among them SW2 SW_Push, SW3 SW_Push, SW4 SW_Push

Commit message: PCB implementation
Parts:
- added R15, R16: 330R, symbol Device:R
- added SW5, SW6: SW_Push, symbol Switch:SW_Push
Connections:
- net +3.3V: now also SW5.1, SW6.1
- net GND: now also R15.2, R16.2
- net COIN_1.5E renamed BTND
- net COIN_1E renamed BTNR
- net COIN_50C renamed BTNL
- new net BTNC: R16.1, SW6.2
- new net BTNU: R15.1, SW5.2
