File: 2. Projects/2. PCB Implementation/PCB design/vending_machine_pcb/FPGA_IO.kicad_sch (KiCad schematic)
At the start: 1 part, among them J2 Conn_01x03_Pin

Commit message: PCB implementation
Parts:
- removed J2: Conn_01x03_Pin, symbol Connector:Conn_01x03_Pin
- added J2: Conn_01x05_Pin, symbol Connector:Conn_01x05_Pin
Connections:
- new net BTNC: J2.1 (Pin_1)
- new net BTND: J2.5 (Pin_5)
- new net BTNL: J2.3 (Pin_3)
- new net BTNR: J2.4 (Pin_4)
- new net BTNU: J2.2 (Pin_2)
Changed lines of the file:
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@@
 	(paper "A4")
+	(junction
+		(at 140.97 54.61)
+		(diameter 0)
+		(color 0 0 0 0)
+	)
 	(junction
 		(at 182.88 74.93)
@@
 	(wire
 		(pts
+			(xy 140.97 52.07) (xy 140.97 54.61)
+		)
+		(stroke
+			(width 0)
+			(type default)
+		)
+	)
+	(wire
+		(pts
 			(xy 73.66 35.56) (xy 27.94 35.56)
 		)
@@
 	(wire
 		(pts
-			(xy 181.61 60.96) (xy 160.02 60.96)
+			(xy 132.08 54.61) (xy 132.08 55.88)
+		)
+		(stroke
+			(width 0)
+			(type default)
+		)
+	)
+	(wire
+		(pts
+			(xy 132.08 55.88) (xy 130.81 55.88)
 		)
 		(stroke
@@
 	(wire
 		(pts
+			(xy 166.37 66.04) (xy 166.37 83.82)
+		)
+		(stroke
+			(width 0)
+			(type default)
+		)
+	)
+	(wire
+		(pts
 			(xy 181.61 59.69) (xy 181.61 60.96)
 		)
@@
 	(wire
 		(pts
+			(xy 130.81 60.96) (xy 181.61 60.96)
+		)
+		(stroke
+			(width 0)
+			(type default)
+		)
+	)
+	(wire
+		(pts
 			(xy 73.66 52.07) (xy 26.67 52.07)
 		)
@@
 	(wire
 		(pts
+			(xy 140.97 54.61) (xy 156.21 54.61)
+		)
+		(stroke
+			(width 0)
+			(type default)
+		)
+	)
+	(wire
+		(pts
 			(xy 231.14 118.11) (xy 232.41 118.11)
 		)
@@
 	(wire
 		(pts
-			(xy 160.02 63.5) (xy 182.88 63.5)
+			(xy 130.81 58.42) (xy 163.83 58.42)
 		)
 		(stroke
@@
 	(wire
 		(pts
+			(xy 130.81 66.04) (xy 166.37 66.04)
+		)
+		(stroke
+			(width 0)
+			(type default)
+		)
+	)
+	(wire
+		(pts
 			(xy 232.41 118.11) (xy 232.41 120.65)
 		)
@@
 	(wire
 		(pts
-			(xy 160.02 58.42) (xy 163.83 58.42)
+			(xy 130.81 63.5) (xy 182.88 63.5)
+		)
+		(stroke
+			(width 0)
+			(type default)
+		)
+	)
+	(wire
+		(pts
+			(xy 132.08 54.61) (xy 140.97 54.61)
 		)
 		(stroke
@@
 		)
 	)
-	(label "COIN_1.5E"
+	(label "BTNR"
 		(at 182.88 83.82 0)
 		(effects
@@
 		)
 	)
-	(label "COIN_50C"
+	(label "BTNU"
 		(at 173.99 54.61 0)
 		(effects
@@
 		)
 	)
+	(label "BTND"
+		(at 166.37 83.82 0)
+		(effects
+			(font
+				(size 1.27 1.27)
+			)
+			(justify left bottom)
+		)
+	)
 	(label "SEG_DP"
 		(at 76.2 115.57 180)
@@
 		)
 	)
+	(label "BTNC"
+		(at 156.21 54.61 0)
+		(effects
+			(font
+				(size 1.27 1.27)
+			)
+			(justify left bottom)
+		)
+	)
 	(label "SEG_B"
 		(at 73.66 35.56 180)
@@
 		)
 	)
-	(label "COIN_1E"
+	(label "BTNL"
 		(at 181.61 58.42 0)
 		(effects
@@
 		)
 	)
+	(hierarchical_label "BTNC"
+		(shape output)
+		(at 140.97 52.07 0)
+		(effects
+			(font
+				(size 1.27 1.27)
+			)
+			(justify left)
+		)
+	)
 	(hierarchical_label "DIG1"
 		(shape output)
@@
 		)
 	)
+	(hierarchical_label "BTND"
+		(shape output)
+		(at 166.37 74.93 0)
+		(effects
+			(font
+				(size 1.27 1.27)
+			)
+			(justify left)
+		)
+	)
 	(hierarchical_label "SEG_C"
 		(shape output)
@@
 		)
 	)
-	(hierarchical_label "COIN_1E"
+	(hierarchical_label "BTNL"
 		(shape output)
 		(at 196.85 59.69 0)
@@
 		)
 	)
-	(hierarchical_label "COIN_50C"
+	(hierarchical_label "BTNU"
 		(shape output)
 		(at 163.83 48.26 0)
@@
 		)
 	)
-	(hierarchical_label "COIN_1.5E"
+	(hierarchical_label "BTNR"
 		(shape output)
 		(at 186.69 74.93 0)
@@
 	)
 	(symbol
-		(lib_id "Connector:Conn_01x03_Pin")
-		(at 154.94 60.96 0)
+		(lib_id "Connector:Conn_01x05_Pin")
+		(at 125.73 60.96 0)
 		(unit 1)
 		(exclude_from_sim no)
@@
 		(fields_autoplaced yes)
 		(property "Reference" "J2"
-			(at 155.575 53.34 0)
+			(at 126.365 50.8 0)
 			(effects
 				(font
@@
 			)
 		)
-		(property "Value" "Conn_01x03_Pin"
-			(at 155.575 55.88 0)
+		(property "Value" "Conn_01x05_Pin"
+			(at 126.365 53.34 0)
 			(effects
 				(font
@@
 		)
 		(property "Footprint" ""
-			(at 154.94 60.96 0)
+			(at 125.73 60.96 0)
 			(effects
 				(font
@@
 		)
 		(property "Datasheet" "~"
-			(at 154.94 60.96 0)
+			(at 125.73 60.96 0)
 			(effects
 				(font
@@
 			)
 		)
-		(property "Description" "Generic connector, single row, 01x03, script generated"
-			(at 154.94 60.96 0)
+		(property "Description" "Generic connector, single row, 01x05, script generated"
+			(at 125.73 60.96 0)
 			(effects
 				(font
@@
 			)
 		)
+		(pin "4"
+		)
 		(pin "1"
 		)
@@
 		(pin "2"
 		)
+		(pin "5"
+		)
 		(instances
