File: 2. Projects/2. PCB Implementation/Coin_Buttons.kicad_sch (KiCad schematic)
At the start: 10 parts, among them SW2 SW_Push, SW3 SW_Push, SW4 SW_Push, SW5 SW_Push, SW6 SW_Push

Commit message: PCB implementation
final design
Parts:
- renumbered SW6 to SW4, SW2 to SW6, SW3 to SW7, SW4 to SW8
Changed lines of the file:
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@@
 		(dnp no)
 		(fields_autoplaced yes)
-		(property "Reference" "SW2"
+		(property "Reference" "SW6"
 			(at 97.79 50.8 0)
 			(effects
@@
 			(project ""
 				(path "/768977ac-7e13-4b05-a33c-a5d6b2881a98/1d7dd153-b5e8-4c52-99fd-a0009788e3fc"
-					(reference "SW2")
+					(reference "SW6")
 					(unit 1)
 				)
@@
 		(dnp no)
 		(fields_autoplaced yes)
-		(property "Reference" "SW6"
+		(property "Reference" "SW4"
 			(at 99.06 19.05 0)
 			(effects
@@
 			(project "vending_machine_pcb"
 				(path "/768977ac-7e13-4b05-a33c-a5d6b2881a98/1d7dd153-b5e8-4c52-99fd-a0009788e3fc"
-					(reference "SW6")
+					(reference "SW4")
 					(unit 1)
 				)
@@
 		(dnp no)
 		(fields_autoplaced yes)
-		(property "Reference" "SW3"
+		(property "Reference" "SW7"
 			(at 95.25 74.93 0)
 			(effects
@@
 			(project ""
 				(path "/768977ac-7e13-4b05-a33c-a5d6b2881a98/1d7dd153-b5e8-4c52-99fd-a0009788e3fc"
-					(reference "SW3")
+					(reference "SW7")
 					(unit 1)
 				)
@@
 		(dnp no)
 		(fields_autoplaced yes)
-		(property "Reference" "SW4"
+		(property "Reference" "SW8"
 			(at 95.25 104.14 0)
 			(effects
@@
 			(project ""
 				(path "/768977ac-7e13-4b05-a33c-a5d6b2881a98/1d7dd153-b5e8-4c52-99fd-a0009788e3fc"
-					(reference "SW4")
-					(unit 1)
-				)
+					(reference "SW8")
+					(unit 1)
+				)
