File: 2. Projects/2. PCB Implementation/Display_interface.kicad_sch (KiCad schematic)
At the start: 17 parts, among them Q1 Q_PNP_EBC, Q2 Q_PNP_EBC, Q3 Q_PNP_EBC, Q4 Q_PNP_EBC, U3 CA56-12EWA

Commit message: PCB implementation
final design
Connections:
- net DIG1 renamed AN0
- net DIG2 renamed AN1
- net DIG3 renamed AN2
- net DIG4 renamed AN3
Changed lines of the file:
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@@
 		)
 	)
-	(label "DIG1"
+	(label "AN0"
 		(at 219.71 64.77 0)
 		(effects
@@
 		)
 	)
-	(label "DIG2"
+	(label "AN1"
 		(at 223.52 106.68 0)
 		(effects
@@
 		)
 	)
-	(label "DIG3"
+	(label "AN2"
 		(at 223.52 149.86 0)
 		(effects
@@
 		)
 	)
-	(label "DIG4"
+	(label "AN3"
 		(at 142.24 124.46 0)
 		(effects
@@
 		)
 	)
-	(hierarchical_label "DIG4"
+	(hierarchical_label "AN3"
 		(shape output)
 		(at 133.35 110.49 0)
@@
 		)
 	)
-	(hierarchical_label "DIG3"
+	(hierarchical_label "AN2"
 		(shape output)
 		(at 228.6 129.54 0)
@@
 		)
 	)
-	(hierarchical_label "DIG2"
+	(hierarchical_label "AN1"
 		(shape output)
 		(at 234.95 86.36 0)
@@
 		)
 	)
-	(hierarchical_label "DIG1"
+	(hierarchical_label "AN0"
 		(shape output)
 		(at 229.87 49.53 0)
