File: 2. Projects/2. PCB Implementation/Power_Supply.kicad_sch (KiCad schematic)
At the start: 12 parts, among them J1 Barrel_Jack, SW1 SW_SPST, U1 LM7805_TO220, U2 LM317_TO-220

Commit message: PCB implementation
final design
Parts:
- renumbered SW1 to SW3
Changed lines of the file:
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@@
 		(dnp no)
 		(fields_autoplaced yes)
-		(property "Reference" "SW1"
+		(property "Reference" "SW3"
 			(at 128.27 22.86 0)
 			(effects
@@
 			(project "vending_machine_pcb"
 				(path "/768977ac-7e13-4b05-a33c-a5d6b2881a98/f50e1eb7-6c81-44e5-a51c-715e81aa5e89"
-					(reference "SW1")
+					(reference "SW3")
 					(unit 1)
 				)
