File: 2. Projects/2. PCB Implementation/vending_machine_pcb.kicad_sch (KiCad schematic)
At the start: 0 parts

Commit message: PCB implementation
final design
Other:
- sheet Display_interface ports: added AN0, AN1, AN2, AN3; removed DIG1, DIG2, DIG3, DIG4
- sheet FPGA_IO ports: added AN0, AN1, AN2, AN3; removed DIG1, DIG2, DIG3, DIG4
Changed lines of the file:
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@@
+	(wire
+		(pts
+			(xy 283.21 26.67) (xy 283.21 105.41)
+		)
+		(stroke
+			(width 0)
+			(type default)
+		)
+	)
+	(wire
+		(pts
+			(xy 261.62 41.91) (xy 276.86 41.91)
+		)
+		(stroke
+			(width 0)
+			(type default)
+		)
+	)
 	(wire
 		(pts
@@
 	(wire
 		(pts
-			(xy 276.86 59.69) (xy 276.86 157.48)
-		)
-		(stroke
-			(width 0)
-			(type default)
-		)
-	)
-	(wire
-		(pts
 			(xy 78.74 176.53) (xy 152.4 176.53)
 		)
@@
 	(wire
 		(pts
+			(xy 280.67 113.03) (xy 261.62 113.03)
+		)
+		(stroke
+			(width 0)
+			(type default)
+		)
+	)
+	(wire
+		(pts
 			(xy 45.72 168.91) (xy 134.62 168.91)
 		)
@@
 	(wire
 		(pts
-			(xy 200.66 151.13) (xy 200.66 161.29)
+			(xy 280.67 31.75) (xy 280.67 113.03)
 		)
 		(stroke
@@
 	(wire
 		(pts
+			(xy 261.62 26.67) (xy 283.21 26.67)
+		)
+		(stroke
+			(width 0)
+			(type default)
+		)
+	)
+	(wire
+		(pts
 			(xy 64.77 102.87) (xy 64.77 172.72)
 		)
@@
 	(wire
 		(pts
-			(xy 226.06 157.48) (xy 226.06 151.13)
-		)
-		(stroke
-			(width 0)
-			(type default)
-		)
-	)
-	(wire
-		(pts
 			(xy 160.02 63.5) (xy 228.6 63.5)
 		)
@@
 	(wire
 		(pts
-			(xy 280.67 48.26) (xy 261.62 48.26)
-		)
-		(stroke
-			(width 0)
-			(type default)
-		)
-	)
-	(wire
-		(pts
-			(xy 180.34 151.13) (xy 180.34 163.83)
+			(xy 271.78 19.05) (xy 271.78 100.33)
+		)
+		(stroke
+			(width 0)
+			(type default)
+		)
+	)
+	(wire
+		(pts
+			(xy 283.21 105.41) (xy 261.62 105.41)
 		)
 		(stroke
@@
 	(wire
 		(pts
+			(xy 276.86 115.57) (xy 261.62 115.57)
+		)
+		(stroke
+			(width 0)
+			(type default)
+		)
+	)
+	(wire
+		(pts
 			(xy 143.51 93.98) (xy 143.51 95.25)
 		)
@@
 	(wire
 		(pts
-			(xy 261.62 72.39) (xy 271.78 72.39)
-		)
-		(stroke
-			(width 0)
-			(type default)
-		)
-	)
-	(wire
-		(pts
 			(xy 255.27 52.07) (xy 255.27 95.25)
 		)
@@
 	(wire
 		(pts
-			(xy 261.62 38.1) (xy 283.21 38.1)
-		)
-		(stroke
-			(width 0)
-			(type default)
-		)
-	)
-	(wire
-		(pts
 			(xy 171.45 52.07) (xy 255.27 52.07)
 		)
@@
 	(wire
 		(pts
-			(xy 283.21 163.83) (xy 180.34 163.83)
+			(xy 261.62 113.03) (xy 261.62 111.76)
+		)
+		(stroke
+			(width 0)
+			(type default)
+		)
+	)
+	(wire
+		(pts
+			(xy 276.86 41.91) (xy 276.86 115.57)
 		)
 		(stroke
@@
 	(wire
 		(pts
+			(xy 261.62 31.75) (xy 280.67 31.75)
+		)
+		(stroke
+			(width 0)
+			(type default)
+		)
+	)
+	(wire
+		(pts
 			(xy 228.6 63.5) (xy 228.6 95.25)
 		)
@@
 	(wire
 		(pts
-			(xy 257.81 151.13) (xy 257.81 154.94)
-		)
-		(stroke
-			(width 0)
-			(type default)
-		)
-	)
-	(wire
-		(pts
 			(xy 152.4 176.53) (xy 152.4 151.13)
 		)
@@
 	(wire
 		(pts
-			(xy 276.86 157.48) (xy 226.06 157.48)
-		)
-		(stroke
-			(width 0)
-			(type default)
-		)
-	)
-	(wire
-		(pts
 			(xy 78.74 102.87) (xy 78.74 176.53)
 		)
@@
 	(wire
 		(pts
-			(xy 200.66 161.29) (xy 280.67 161.29)
-		)
-		(stroke
-			(width 0)
-			(type default)
-		)
-	)
-	(wire
-		(pts
 			(xy 143.51 172.72) (xy 143.51 151.13)
 		)
@@
 	(wire
 		(pts
-			(xy 261.62 59.69) (xy 276.86 59.69)
-		)
-		(stroke
-			(width 0)
-			(type default)
-		)
-	)
-	(wire
-		(pts
-			(xy 271.78 154.94) (xy 271.78 72.39)
+			(xy 250.19 19.05) (xy 271.78 19.05)
 		)
 		(stroke
@@
 	(wire
 		(pts
-			(xy 257.81 154.94) (xy 271.78 154.94)
-		)
-		(stroke
-			(width 0)
-			(type default)
-		)
-	)
-	(wire
-		(pts
-			(xy 283.21 38.1) (xy 283.21 163.83)
-		)
-		(stroke
-			(width 0)
-			(type default)
-		)
-	)
-	(wire
-		(pts
-			(xy 280.67 161.29) (xy 280.67 48.26)
+			(xy 250.19 21.59) (xy 250.19 19.05)
+		)
+		(stroke
+			(width 0)
+			(type default)
+		)
+	)
+	(wire
+		(pts
+			(xy 271.78 100.33) (xy 261.62 100.33)
 		)
 		(stroke
@@
 			)
 		)
-		(pin "DIG1" output
-			(at 180.34 151.13 270)
-			(effects
-				(font
-					(size 1.27 1.27)
-				)
-				(justify left)
-			)
-		)
-		(pin "DIG2" output
-			(at 200.66 151.13 270)
-			(effects
-				(font
-					(size 1.27 1.27)
-				)
-				(justify left)
-			)
-		)
-		(pin "DIG3" output
-			(at 226.06 151.13 270)
-			(effects
-				(font
-					(size 1.27 1.27)
-				)
-				(justify left)
-			)
-		)
-		(pin "DIG4" output
-			(at 257.81 151.13 270)
-			(effects
-				(font
-					(size 1.27 1.27)
-				)
-				(justify left)
-			)
-		)
 		(pin "BTNC" output
 			(at 127 151.13 270)
@@
 				)
 				(justify left)
+			)
+		)
+		(pin "AN1" output
+			(at 261.62 105.41 0)
+			(effects
+				(font
+					(size 1.27 1.27)
+				)
+				(justify right)
+			)
+		)
+		(pin "AN2" output
+			(at 261.62 111.76 0)
+			(effects
+				(font
+					(size 1.27 1.27)
+				)
+				(justify right)
+			)
+		)
+		(pin "AN3" output
+			(at 261.62 115.57 0)
+			(effects
+				(font
+					(size 1.27 1.27)
+				)
+				(justify right)
+			)
+		)
+		(pin "AN0" output
+			(at 261.62 100.33 0)
+			(effects
+				(font
+					(size 1.27 1.27)
+				)
+				(justify right)
 			)
 		)
@@
 			)
 		)
-		(pin "DIG1" output
-			(at 261.62 38.1 0)
-			(effects
-				(font
-					(size 1.27 1.27)
-				)
-				(justify right)
-			)
-		)
-		(pin "DIG2" output
-			(at 261.62 48.26 0)
-			(effects
-				(font
-					(size 1.27 1.27)
-				)
-				(justify right)
-			)
-		)
-		(pin "DIG3" output
-			(at 261.62 59.69 0)
-			(effects
-				(font
-					(size 1.27 1.27)
-				)
-				(justify right)
-			)
-		)
-		(pin "DIG4" output
-			(at 261.62 72.39 0)
-			(effects
-				(font
+		(pin "AN1" output
+			(at 261.62 26.67 0)
+			(effects
+				(font
+					(size 1.27 1.27)
+				)
+				(justify right)
+			)
+		)
+		(pin "AN2" output
+			(at 261.62 31.75 0)
+			(effects
+				(font
+					(size 1.27 1.27)
+				)
+				(justify right)
+			)
+		)
+		(pin "AN3" output
+			(at 261.62 41.91 0)
+			(effects
+				(font
+					(size 1.27 1.27)
+				)
+				(justify right)
+			)
+		)
+		(pin "AN0" output
+			(at 250.19 21.59 90)
+			(effects
+				(font
