File: 2. Projects/5. PCB Implementation/FPGA_IO.kicad_sch (KiCad schematic)
At the start: 5 parts, among them J2 Conn_01x05_Pin, J3 Conn_01x30

Commit message: UPDATED Fpga model
Parts:
- removed J3: Conn_01x30, symbol Connector_Generic:Conn_01x30
- added BaseResistor5, BaseResistor6, BaseResistor7, BaseResistor8: 1kR, Resistor_THT:R_Axial_DIN0204_L3.6mm_D1.6mm_P5.08mm_Vertical, symbol Device:R
- added Cin3: 100n, Capacitor_THT:C_Axial_L3.8mm_D2.6mm_P10.00mm_Horizontal, symbol Device:C
- added Cin4: 1u, Capacitor_THT:C_Axial_L3.8mm_D2.6mm_P7.50mm_Horizontal, symbol Device:C
- added Cout3: 100n, Capacitor_THT:CP_Axial_L10.0mm_D6.0mm_P15.00mm_Horizontal, symbol Device:C
- added Cout4: 10u, Capacitor_THT:CP_Axial_L10.0mm_D6.0mm_P15.00mm_Horizontal, symbol Device:C
- added D2: PWR_LED, LED_THT:LED_D3.0mm, symbol Device:LED
- added J3: Barrel_Jack, Connector_BarrelJack:BarrelJack_CLIFF_FC681465S_SMT_Horizontal, symbol Connector:Barrel_Jack
- added Q5, Q6, Q7, Q8: Q_PNP_EBC, Package_TO_SOT_THT:TO-92, symbol Transistor_BJT:Q_PNP_EBC
- added R20, R21, R22: 330R, Resistor_THT:R_Axial_DIN0204_L3.6mm_D1.6mm_P5.08mm_Vertical, symbol Device:R
- added R23, R24, R25, R26, R27, R28, R29, R30, R31, R32, R33: 330R, Resistor_THT:R_Axial_DIN0204_L3.6mm_D1.6mm_P5.08mm_Horizontal, symbol Device:R
- added R34: 240R, Resistor_THT:R_Axial_DIN0204_L3.6mm_D1.6mm_P5.08mm_Horizontal, symbol Device:R
- added R35: 390R, Resistor_THT:R_Axial_DIN0204_L3.6mm_D1.6mm_P1.90mm_Vertical, symbol Device:R
- added SW1, SW10, SW11, SW2, SW9: SW_Push, Button_Switch_Keyboard:SW_Cherry_MX_1.00u_PCB, symbol Switch:SW_Push
- added SW12: SW_SPST, Button_Switch_Keyboard:SW_Cherry_MX_1.00u_PCB, symbol Switch:SW_SPST
- added U4: XC7A100T-CSG324, Package_BGA:BGA-324_15x15mm_Layout18x18_P0.8mm, symbol FPGA_Xilinx_Artix7:XC7A100T-CSG324
- added U5: CA56-12EWA, Display_7Segment:CA56-12EWA, symbol Display_Character:CA56-12EWA
- added U6: LM7805_TO220, Package_TO_SOT_THT:TO-220-3_Vertical, symbol Regulator_Linear:LM7805_TO220
- added U7: LM317_TO-220, Package_TO_SOT_THT:TO-220-3_Vertical, symbol Regulator_Linear:LM317_TO-220
- J2: footprint (none) -> Connector_PinHeader_2.54mm:PinHeader_1x05_P2.54mm_Vertical_SMD_Pin1Left
- R17, R19: footprint (none) -> Resistor_THT:R_Axial_DIN0204_L3.6mm_D1.6mm_P5.08mm_Vertical
- R18: footprint (none) -> Resistor_THT:R_Axial_DIN0204_L3.6mm_D1.6mm_P7.62mm_Horizontal
Connections:
- net AN0: now also BaseResistor6.1, BaseResistor6.2, Q6.2 (B), U4.E3 (IO_0_14), U4.G10 (IO_L23P_T3_FOE_B_15)
- net AN1: now also BaseResistor7.1, BaseResistor7.2, Q7.2 (B), U4.N2 (IO_L23N_T3_A02_D18_14), U4.P13 (IO_L23N_T3_FWE_B_15)
- net AN2: now also BaseResistor8.1, BaseResistor8.2, Q8.2 (B), U4.B4 (IO_L5P_T0_D06_14), U4.J4 (IO_L24P_T3_A01_D17_14)
- net AN3: now also BaseResistor5.1, BaseResistor5.2, Q5.2 (B), U4.G11 (IO_L19P_T3_A22_15), U4.L6 (IO_L23P_T3_A03_D19_14)
- net BTNC: now also R30.1, SW10.2, U4.M5 (IO_L9P_T1_DQS_14)
- net BTND: now also R32.1, SW2.2, U4.N10 (IO_L9N_T1_DQS_D13_14)
- net BTNL: now also R28.1, SW9.2, U4.M11 (IO_L12P_T1_MRCC_14)
- net BTNR: now also R29.1, SW1.2, U4.T4 (IO_L10N_T1_D15_14)
- net BTNU: now also R31.1, SW11.2, U4.A3 (IO_L4N_T0_D05_14)
- net GND: now also Cin3.2, Cin4.2, Cout3.2, Cout4.2, D2.1 (K), J3.2, R29.2, R32.2, R35.2, U4.F7 (IO_L16P_T2_A28_15), U4.H13 (IO_0_15), U6.2 (GND)
- net LED0: now also U4.F2 (IO_L18P_T2_A24_15)
- net LED1: now also U4.A4 (IO_L24P_T3_RS1_15)
- net LED2: now also U4.J2 (IO_L21P_T3_DQS_14)
- net SEG_A: now also R24.1, R24.2, U4.D8 (IO_L1P_T0_D00_MOSI_14), U4.F12 (IO_L24N_T3_A00_D16_14), U5.11 (a)
- net SEG_B: now also R26.1, R26.2, U4.H2 (IO_25_14), U4.N9 (IO_L1N_T0_D01_DIN_14), U5.7 (b)
- net SEG_C: now also R20.1, R20.2, U4.J5 (IO_25_15), U4.K2 (IO_L17P_T2_A26_15), U4.L10 (IO_L2P_T0_D02_14), U5.4 (c)
- net SEG_D: now also R21.1, R21.2, R22.1, R22.2, R25.1, R25.2, R27.1, R27.2, U4.B5 (IO_L4P_T0_D04_14), U4.F1 (IO_L13P_T2_MRCC_14), U4.G12 (IO_L2N_T0_D03_14), U4.G6 (IO_L10P_T1_D14_14), U4.G7 (IO_L5N_T0_D07_14), U4.J11 (IO_L7N_T1_D10_14), U4.M10 (IO_L19N_T3_A21_VREF_15), U5.1 (e), U5.2 (d), U5.3 (DPX), U5.5 (g)
- net SEG_F: now also R23.1, R23.2, U4.E10 (IO_L19P_T3_A10_D26_14), U4.F3 (IO_L8N_T1_D12_14), U5.10 (f)
- net SW0: now also U4.E6 (IO_L18N_T2_A11_D27_14)
- net SW1: now also U4.M2 (IO_L17P_T2_A14_D30_14)
- net SW2: now also U4.M4 (IO_L20N_T3_A19_15)
- new net: D2.2 (A), R33.1
- new net: R34.1, R35.1, U7.1 (ADJ)
- new net: Cin4.1, U7.3 (VI)
- new net: Q6.3 (C), U5.12 (CA1)
- new net: Q7.3 (C), U5.9 (CA2)
- new net: Q5.3 (C), U5.6 (CA4)
- new net: Q8.3 (C), U5.8 (CA3)
- new net +3.3V: SW1.1, SW10.1, SW11.1, SW2.1, SW9.1, U4.B7 (IO_L20P_T3_A08_D24_14), U4.F6 (IO_L20N_T3_A07_D23_14), U4.M6 (IO_L17N_T2_A13_D29_14), U4.N5 (IO_L16N_T2_A15_D31_14), U4.R4 (IO_L18P_T2_A12_D28_14)
- new net +3v3: Cout4.1, R28.2, R30.2, R31.2, R34.2, SW12.2 (B), U4.A12 (VCCO_14), U4.A9 (VCCO_14), U4.E2 (VCCO_14), U4.E4 (VCCO_15), U4.F11 (VCCO_14), U4.G5 (VCCO_15), U4.H3 (VCCO_14), U4.V4 (VCCO_14), U7.2 (VO)
- new net +5V: Cout3.1, Q5.1 (E), Q6.1 (E), Q7.1 (E), Q8.1 (E), R33.2, U6.3 (VO)
- new net Vin: Cin3.1, J3.1, SW12.1 (A), U6.1 (VI)
- no-connect marks 7 -> 58
Other:
- note added: "Vout = 1.25V × (1 + R2/R1) ≈ 3.3V"
- note added: "When FPGA drives DIGx LOW: PNP turns ON +5V flows to the digit (e.g., CA1) When DIGx is HIGH (or unconnected): PNP turns OFF No current flows → digit off"
- note added: "limit current from FPGA"
- moved on the sheet: J2, R17, R18, R19
