File: 2. Projects/5. PCB Implementation/_autosave-vending_machine_pcb.kicad_pcb (KiCad board)
At the start: 2 copper layers, 3 parts, among them U1 LM7805_TO220, U2 LM317_TO-220, U3 CA56-12EWA

Commit message: UPDATED Fpga model
Parts:
- added BaseResistor1: 1kR, Resistor_THT:R_Axial_DIN0204_L3.6mm_D1.6mm_P2.54mm_Vertical, F.Cu at (27.9, 41.9)
- added BaseResistor2: 1kR, Resistor_THT:R_Axial_DIN0204_L3.6mm_D1.6mm_P2.54mm_Vertical, F.Cu at (24.1, 49.5)
- added BaseResistor3: 1kR, Resistor_THT:R_Axial_DIN0204_L3.6mm_D1.6mm_P1.90mm_Vertical, F.Cu at (25.8, 48.4)
- added BaseResistor4: 1kR, Resistor_THT:R_Axial_DIN0204_L3.6mm_D1.6mm_P5.08mm_Horizontal, F.Cu at (16.5, 35.6)
- added BaseResistor5: 1kR, Resistor_THT:R_Axial_DIN0204_L3.6mm_D1.6mm_P5.08mm_Vertical, F.Cu at (16.6, 30.5)
- added BaseResistor6: 1kR, Resistor_THT:R_Axial_DIN0204_L3.6mm_D1.6mm_P5.08mm_Vertical, F.Cu at (12.7, 44.5)
- added BaseResistor7: 1kR, Resistor_THT:R_Axial_DIN0204_L3.6mm_D1.6mm_P5.08mm_Vertical, F.Cu at (12.7, 47.6)
- added BaseResistor8: 1kR, Resistor_THT:R_Axial_DIN0204_L3.6mm_D1.6mm_P5.08mm_Vertical, F.Cu at (12.7, 50.8)
- added Cin1: 100n, Capacitor_THT:C_Axial_L3.8mm_D2.6mm_P7.50mm_Horizontal, F.Cu at (13.1, 48.9)
- added Cin2: 1u, Capacitor_THT:C_Axial_L3.8mm_D2.6mm_P7.50mm_Horizontal, F.Cu at (13.1, 53.1)
- added Cin3: 100n, Capacitor_THT:C_Axial_L3.8mm_D2.6mm_P10.00mm_Horizontal, F.Cu at (26.8, 30.5)
- added Cin4: 1u, Capacitor_THT:C_Axial_L3.8mm_D2.6mm_P7.50mm_Horizontal, F.Cu at (13.1, 42.8)
- added Cout1: 100n, Capacitor_THT:CP_Axial_L10.0mm_D6.0mm_P15.00mm_Horizontal, F.Cu at (256.5, 163.8)
- added Cout2: 10u, Capacitor_THT:CP_Axial_L10.0mm_D6.0mm_P15.00mm_Horizontal, F.Cu at (227.6, 134.2)
- added Cout3: 100n, Capacitor_THT:CP_Axial_L10.0mm_D6.0mm_P15.00mm_Horizontal, F.Cu at (174.3, 99.0)
- added Cout4: 10u, Capacitor_THT:CP_Axial_L10.0mm_D6.0mm_P15.00mm_Horizontal, F.Cu at (265.6, 77.5)
- added D1: PWR_LED, LED_THT:LED_D3.0mm, F.Cu at (78.0, 120.5)
- added D2: PWR_LED, LED_THT:LED_D3.0mm, F.Cu at (64.5, 130.3)
- added J1: Barrel_Jack, Connector_BarrelJack:BarrelJack_CLIFF_FC681465S_SMT_Horizontal, F.Cu at (234.8, 146.0)
- added J2: Conn_01x05_Pin, Connector_PinHeader_2.54mm:PinHeader_1x05_P2.54mm_Vertical_SMD_Pin1Left, F.Cu at (260.4, 82.5)
- added J3: Barrel_Jack, Connector_BarrelJack:BarrelJack_CLIFF_FC681465S_SMT_Horizontal, F.Cu at (242.9, 102.8)
- added Q1: Q_PNP_EBC, Package_TO_SOT_THT:TO-92, F.Cu at (78.3, 95.8)
- added Q2: Q_PNP_EBC, Package_TO_SOT_THT:TO-92, F.Cu at (78.3, 101.6)
- added Q3: Q_PNP_EBC, Package_TO_SOT_THT:TO-92, F.Cu at (78.3, 107.4)
- added Q4: Q_PNP_EBC, Package_TO_SOT_THT:TO-92, F.Cu at (78.3, 113.2)
- added Q5: Q_PNP_EBC, Package_TO_SOT_THT:TO-92, F.Cu at (64.8, 95.8)
- added Q6: Q_PNP_EBC, Package_TO_SOT_THT:TO-92, F.Cu at (64.8, 101.6)
- added Q7: Q_PNP_EBC, Package_TO_SOT_THT:TO-92, F.Cu at (64.8, 107.4)
- added Q8: Q_PNP_EBC, Package_TO_SOT_THT:TO-92, F.Cu at (64.8, 113.2)
- added R1: 240R, Resistor_THT:R_Axial_DIN0204_L3.6mm_D1.6mm_P1.90mm_Vertical, F.Cu at (179.4, 158.8)
- added R10: 330R, Resistor_THT:R_Axial_DIN0204_L3.6mm_D1.6mm_P5.08mm_Vertical, F.Cu at (196.3, 149.9)
- added R11: 330R, Resistor_THT:R_Axial_DIN0204_L3.6mm_D1.6mm_P7.62mm_Horizontal, F.Cu at (204.3, 137.3)
- added R12: 330R, Resistor_THT:R_Axial_DIN0204_L3.6mm_D1.6mm_P5.08mm_Horizontal, F.Cu at (217.2, 78.7)
- added R13: 330R, Resistor_THT:R_Axial_DIN0204_L3.6mm_D1.6mm_P5.08mm_Vertical, F.Cu at (217.3, 66.1)
- added R14: 330R, Resistor_THT:R_Axial_DIN0204_L3.6mm_D1.6mm_P5.08mm_Vertical, F.Cu at (217.3, 69.3)
- added R15: 330R, Resistor_THT:R_Axial_DIN0204_L3.6mm_D1.6mm_P5.08mm_Vertical, F.Cu at (217.3, 72.4)
- added R16: 330R, Resistor_THT:R_Axial_DIN0204_L3.6mm_D1.6mm_P5.08mm_Vertical, F.Cu at (217.3, 75.6)
- added R17: R, Resistor_THT:R_Axial_DIN0204_L3.6mm_D1.6mm_P5.08mm_Vertical, F.Cu at (166.0, 96.8)
- added R18: R, Resistor_THT:R_Axial_DIN0204_L3.6mm_D1.6mm_P7.62mm_Horizontal, F.Cu at (204.3, 124.2)
- added R19: R, Resistor_THT:R_Axial_DIN0204_L3.6mm_D1.6mm_P5.08mm_Vertical, F.Cu at (166.0, 99.9)
- added R2: 390R, Resistor_THT:R_Axial_DIN0204_L3.6mm_D1.6mm_P2.54mm_Vertical, F.Cu at (173.8, 158.8)
- added R20: 330R, Resistor_THT:R_Axial_DIN0204_L3.6mm_D1.6mm_P5.08mm_Vertical, F.Cu at (166.0, 103.0)
- added R21: 330R, Resistor_THT:R_Axial_DIN0204_L3.6mm_D1.6mm_P5.08mm_Vertical, F.Cu at (180.0, 136.9)
- added R22: 330R, Resistor_THT:R_Axial_DIN0204_L3.6mm_D1.6mm_P5.08mm_Vertical, F.Cu at (180.0, 140.1)
- added R23: 330R, Resistor_THT:R_Axial_DIN0204_L3.6mm_D1.6mm_P5.08mm_Horizontal, F.Cu at (227.3, 66.1)
- added R24: 330R, Resistor_THT:R_Axial_DIN0204_L3.6mm_D1.6mm_P5.08mm_Horizontal, F.Cu at (227.3, 69.3)
- added R25: 330R, Resistor_THT:R_Axial_DIN0204_L3.6mm_D1.6mm_P5.08mm_Horizontal, F.Cu at (227.3, 72.4)
- added R26: 330R, Resistor_THT:R_Axial_DIN0204_L3.6mm_D1.6mm_P5.08mm_Horizontal, F.Cu at (227.3, 75.6)
- added R27: 330R, Resistor_THT:R_Axial_DIN0204_L3.6mm_D1.6mm_P5.08mm_Horizontal, F.Cu at (227.3, 78.7)
- added R28: 330R, Resistor_THT:R_Axial_DIN0204_L3.6mm_D1.6mm_P5.08mm_Horizontal, F.Cu at (227.3, 81.9)
- added R29: 330R, Resistor_THT:R_Axial_DIN0204_L3.6mm_D1.6mm_P5.08mm_Horizontal, F.Cu at (227.3, 85.0)
- added R3: 330R, Resistor_THT:R_Axial_DIN0204_L3.6mm_D1.6mm_P5.08mm_Horizontal, F.Cu at (173.7, 155.6)
- added R30: 330R, Resistor_THT:R_Axial_DIN0204_L3.6mm_D1.6mm_P5.08mm_Horizontal, F.Cu at (227.3, 88.2)
- added R31: 330R, Resistor_THT:R_Axial_DIN0204_L3.6mm_D1.6mm_P5.08mm_Horizontal, F.Cu at (227.3, 91.3)
- added R32: 330R, Resistor_THT:R_Axial_DIN0204_L3.6mm_D1.6mm_P5.08mm_Horizontal, F.Cu at (227.3, 94.5)
- added R33: 330R, Resistor_THT:R_Axial_DIN0204_L3.6mm_D1.6mm_P5.08mm_Horizontal, F.Cu at (227.3, 97.6)
- added R34: 240R, Resistor_THT:R_Axial_DIN0204_L3.6mm_D1.6mm_P5.08mm_Horizontal, F.Cu at (227.3, 100.8)
- added R35: 390R, Resistor_THT:R_Axial_DIN0204_L3.6mm_D1.6mm_P1.90mm_Vertical, F.Cu at (204.4, 121.1)
- added R4: 330R, Resistor_THT:R_Axial_DIN0204_L3.6mm_D1.6mm_P5.08mm_Vertical, F.Cu at (196.3, 134.2)
- added R5: 330R, Resistor_THT:R_Axial_DIN0204_L3.6mm_D1.6mm_P5.08mm_Vertical, F.Cu at (196.3, 137.3)
- added R6: 330R, Resistor_THT:R_Axial_DIN0204_L3.6mm_D1.6mm_P7.62mm_Horizontal, F.Cu at (204.3, 134.2)
- added R7: 330R, Resistor_THT:R_Axial_DIN0204_L3.6mm_D1.6mm_P5.08mm_Vertical, F.Cu at (196.3, 140.4)
- added R8: 330R, Resistor_THT:R_Axial_DIN0204_L3.6mm_D1.6mm_P5.08mm_Vertical, F.Cu at (196.3, 143.6)
- added R9: 330R, Resistor_THT:R_Axial_DIN0204_L3.6mm_D1.6mm_P5.08mm_Vertical, F.Cu at (196.3, 146.8)
- added SW1: SW_Push, Button_Switch_Keyboard:SW_Cherry_MX_1.00u_PCB, F.Cu at (157.8, 67.5)
- added SW10: SW_Push, Button_Switch_Keyboard:SW_Cherry_MX_1.00u_PCB, F.Cu at (172.9, 82.5)
- added SW11: SW_Push, Button_Switch_Keyboard:SW_Cherry_MX_1.00u_PCB, F.Cu at (188.0, 67.5)
- added SW12: SW_SPST, Button_Switch_Keyboard:SW_Cherry_MX_1.00u_PCB, F.Cu at (188.0, 82.5)
- added SW2: SW_Push, Button_Switch_Keyboard:SW_Cherry_MX_1.00u_PCB, F.Cu at (157.8, 82.5)
- added SW3: SW_SPST, Button_Switch_Keyboard:SW_Cherry_MX_1.00u_PCB, F.Cu at (158.8, 181.6)
- added SW4: SW_Push, Button_Switch_Keyboard:SW_Cherry_MX_1.00u_PCB, F.Cu at (154.9, 22.9)
- added SW5: SW_Push, Button_Switch_Keyboard:SW_Cherry_MX_1.00u_PCB, F.Cu at (135.9, 39.5)
- added SW6: SW_Push, Button_Switch_Keyboard:SW_Cherry_MX_1.00u_PCB, F.Cu at (135.9, 54.6)
- added SW7: SW_Push, Button_Switch_Keyboard:SW_Cherry_MX_1.00u_PCB, F.Cu at (135.9, 69.7)
- added SW8: SW_Push, Button_Switch_Keyboard:SW_Cherry_MX_1.00u_PCB, F.Cu at (135.9, 84.8)
- added SW9: SW_Push, Button_Switch_Keyboard:SW_Cherry_MX_1.00u_PCB, F.Cu at (172.9, 67.5)
- added U4: XC7A100T-CSG324, Package_BGA:BGA-324_15x15mm_Layout18x18_P0.8mm, F.Cu at (198.3, 125.0)
- added U5: CA56-12EWA, Display_7Segment:CA56-12EWA, F.Cu at (19.1, 162.6)
- added U6: LM7805_TO220, Package_TO_SOT_THT:TO-220-3_Vertical, F.Cu at (66.0, 119.6)
- added U7: LM317_TO-220, Package_TO_SOT_THT:TO-220-3_Vertical, F.Cu at (66.0, 125.6)
- moved U3 79.2 mm to (111.9, 161.3)
- moved U2 49.0 mm to (166.4, 121.4)
- moved U1 49.0 mm to (166.4, 108.0)
Connections:
- U3 pad 1: /Display_interface/SEG_E -> /Display_interface/SEG_D
- U3 pad 3: /Display_interface/SEG_DP -> /Display_interface/SEG_D
- U3 pad 5: /Display_interface/SEG_G -> /Display_interface/SEG_D
