File: 2. Projects/4. PCB Prototyping/_autosave-vending_machine_pcb.kicad_pcb (KiCad board)
At the start: 2 copper layers, 83 parts, among them J1 Barrel_Jack, J2 Conn_01x05_Pin, J3 Barrel_Jack, Q1 Q_PNP_EBC, Q2 Q_PNP_EBC, Q3 Q_PNP_EBC, Q4 Q_PNP_EBC, Q5 Q_PNP_EBC, Q6 Q_PNP_EBC, Q7 Q_PNP_EBC, Q8 Q_PNP_EBC, SW1 SW_Push, SW10 SW_Push, SW11 SW_Push, SW12 SW_SPST, SW2 SW_Push, SW3 SW_SPST, SW4 SW_Push, SW5 SW_Push, SW6 SW_Push, SW7 SW_Push, SW8 SW_Push, SW9 SW_Push, U1 LM7805_TO220, U2 LM317_TO-220, U3 CA56-12EWA, U4 XC7A100T-CSG324, U5 CA56-12EWA, U6 LM7805_TO220, U7 LM317_TO-220

Commit message: final project files
including FPGA, PCB layout, BOM, Garber zip files
Parts:
- removed BaseResistor1, BaseResistor2: 1kR, Resistor_THT:R_Axial_DIN0204_L3.6mm_D1.6mm_P2.54mm_Vertical
- removed BaseResistor3: 1kR, Resistor_THT:R_Axial_DIN0204_L3.6mm_D1.6mm_P1.90mm_Vertical
- removed BaseResistor4: 1kR, Resistor_THT:R_Axial_DIN0204_L3.6mm_D1.6mm_P5.08mm_Horizontal
- removed BaseResistor5, BaseResistor6, BaseResistor7, BaseResistor8: 1kR, Resistor_THT:R_Axial_DIN0204_L3.6mm_D1.6mm_P5.08mm_Vertical
- removed Cin1: 100n, Capacitor_THT:C_Axial_L3.8mm_D2.6mm_P7.50mm_Horizontal
- removed Cin2, Cin4: 1u, Capacitor_THT:C_Axial_L3.8mm_D2.6mm_P7.50mm_Horizontal
- removed Cin3: 100n, Capacitor_THT:C_Axial_L3.8mm_D2.6mm_P10.00mm_Horizontal
- removed Cout1, Cout3: 100n, Capacitor_THT:CP_Axial_L10.0mm_D6.0mm_P15.00mm_Horizontal
- removed Cout2, Cout4: 10u, Capacitor_THT:CP_Axial_L10.0mm_D6.0mm_P15.00mm_Horizontal
- added C1: C, Capacitor_SMD:C_0603_1608Metric, F.Cu at (201.7, 180.0)
- added C2: C, Capacitor_SMD:C_0603_1608Metric, F.Cu at (201.7, 182.6)
- added C3: C, Capacitor_SMD:C_0603_1608Metric, F.Cu at (201.7, 185.1)
- added C4: C, Capacitor_SMD:C_0603_1608Metric, F.Cu at (201.7, 187.6)
- added C5: C, Capacitor_SMD:C_0603_1608Metric, F.Cu at (220.9, 134.7)
- added C6: C, Capacitor_SMD:C_0603_1608Metric, F.Cu at (220.9, 137.2)
- added C7: C, Capacitor_SMD:C_0603_1608Metric, F.Cu at (220.9, 139.8)
- added C8: C, Capacitor_SMD:C_0603_1608Metric, F.Cu at (220.9, 142.3)
- added R36: R, Resistor_THT:R_Axial_DIN0207_L6.3mm_D2.5mm_P2.54mm_Vertical, F.Cu at (266.5, 132.4)
- added R37: R, Resistor_THT:R_Axial_DIN0207_L6.3mm_D2.5mm_P2.54mm_Vertical, F.Cu at (266.5, 136.4)
- added R38: R, Resistor_THT:R_Axial_DIN0207_L6.3mm_D2.5mm_P2.54mm_Vertical, F.Cu at (266.5, 140.5)
- added R39: R, Resistor_THT:R_Axial_DIN0207_L6.3mm_D2.5mm_P2.54mm_Vertical, F.Cu at (182.1, 168.2)
- added R40: R, Resistor_THT:R_Axial_DIN0207_L6.3mm_D2.5mm_P2.54mm_Vertical, F.Cu at (182.1, 172.2)
- added R41: R, Resistor_THT:R_Axial_DIN0207_L6.3mm_D2.5mm_P2.54mm_Vertical, F.Cu at (182.1, 176.3)
- added R42: R, Resistor_THT:R_Axial_DIN0207_L6.3mm_D2.5mm_P2.54mm_Vertical, F.Cu at (182.1, 180.3)
- added R43: R, Resistor_THT:R_Axial_DIN0207_L6.3mm_D2.5mm_P2.54mm_Vertical, F.Cu at (182.1, 184.4)
- D1, D2: value PWR_LED -> LED; footprint LED_THT:LED_D3.0mm -> LED_SMD:LED-APA102-2020
- J1, J3: footprint Connector_BarrelJack:BarrelJack_CLIFF_FC681465S_SMT_Horizontal -> Connector_BarrelJack:BarrelJack_Horizontal
- J2: footprint Connector_PinHeader_2.54mm:PinHeader_1x05_P2.54mm_Vertical_SMD_Pin1Left -> Connector_PinSocket_1.00mm:PinSocket_1x05_P1.00mm_Vertical_SMD_Pin1Left
- Q1, Q2, Q3, Q4, Q5, Q6, Q7, Q8: footprint Package_TO_SOT_THT:TO-92 -> Package_TO_SOT_SMD:SOT-23
- R1: value 240R -> R; footprint Resistor_THT:R_Axial_DIN0204_L3.6mm_D1.6mm_P1.90mm_Vertical -> Resistor_THT:R_Axial_DIN0207_L6.3mm_D2.5mm_P2.54mm_Vertical
- R10, R13, R14, R15, R16, R20, R21, R22, R4, R5, R7, R8, R9: value 330R -> R; footprint Resistor_THT:R_Axial_DIN0204_L3.6mm_D1.6mm_P5.08mm_Vertical -> Resistor_THT:R_Axial_DIN0207_L6.3mm_D2.5mm_P2.54mm_Vertical
- R11, R6: value 330R -> R; footprint Resistor_THT:R_Axial_DIN0204_L3.6mm_D1.6mm_P7.62mm_Horizontal -> Resistor_THT:R_Axial_DIN0207_L6.3mm_D2.5mm_P2.54mm_Vertical
- R12, R23, R24, R25, R26, R27, R28, R29, R3, R30, R31, R32, R33: value 330R -> R; footprint Resistor_THT:R_Axial_DIN0204_L3.6mm_D1.6mm_P5.08mm_Horizontal -> Resistor_THT:R_Axial_DIN0207_L6.3mm_D2.5mm_P2.54mm_Vertical
- R17, R19: footprint Resistor_THT:R_Axial_DIN0204_L3.6mm_D1.6mm_P5.08mm_Vertical -> Resistor_THT:R_Axial_DIN0207_L6.3mm_D2.5mm_P2.54mm_Vertical
- R18: footprint Resistor_THT:R_Axial_DIN0204_L3.6mm_D1.6mm_P7.62mm_Horizontal -> Resistor_THT:R_Axial_DIN0207_L6.3mm_D2.5mm_P2.54mm_Vertical
- R2: value 390R -> R; footprint Resistor_THT:R_Axial_DIN0204_L3.6mm_D1.6mm_P2.54mm_Vertical -> Resistor_THT:R_Axial_DIN0207_L6.3mm_D2.5mm_P2.54mm_Vertical
- R34: value 240R -> R; footprint Resistor_THT:R_Axial_DIN0204_L3.6mm_D1.6mm_P5.08mm_Horizontal -> Resistor_THT:R_Axial_DIN0207_L6.3mm_D2.5mm_P2.54mm_Vertical
- R35: value 390R -> R; footprint Resistor_THT:R_Axial_DIN0204_L3.6mm_D1.6mm_P1.90mm_Vertical -> Resistor_THT:R_Axial_DIN0207_L6.3mm_D2.5mm_P2.54mm_Vertical
- SW1, SW7: value SW_Push -> SW_SPST; footprint Button_Switch_Keyboard:SW_Cherry_MX_1.00u_PCB -> Button_Switch_THT:SW_PUSH_6mm_H13mm
- SW10, SW11, SW2, SW4, SW5, SW6, SW8, SW9: footprint Button_Switch_Keyboard:SW_Cherry_MX_1.00u_PCB -> Button_Switch_THT:SW_PUSH_6mm_H13mm
- SW12, SW3: value SW_SPST -> SW_Push; footprint Button_Switch_Keyboard:SW_Cherry_MX_1.00u_PCB -> Button_Switch_THT:SW_PUSH_6mm_H13mm
- U5: value CA56-12EWA -> LM7805_TO220; footprint Display_7Segment:CA56-12EWA -> Package_TO_SOT_THT:TO-220-3_Vertical
- U6: value LM7805_TO220 -> LM317_TO-220
- U7: value LM317_TO-220 -> CA56-12EWA; footprint Package_TO_SOT_THT:TO-220-3_Vertical -> Display_7Segment:CA56-12EWA
- moved U5 202.2 mm to (221.1, 155.5)
- moved Q5 190.9 mm to (255.2, 109.2)
- moved Q6 190.9 mm to (255.2, 113.9)
- moved Q7 190.8 mm to (255.2, 118.5)
- moved Q8 190.7 mm to (255.2, 123.1)
- moved U7 168.9 mm to (234.9, 126.4)
- moved Q1 164.2 mm to (242.4, 102.4)
- moved U6 160.6 mm to (221.1, 161.4)
- moved D2 157.2 mm to (220.9, 145.6)
- moved Q2 150.3 mm to (227.9, 116.2)
- moved Q3 150.2 mm to (227.9, 120.8)
- moved Q4 150.1 mm to (227.9, 125.5)
- moved D1 145.2 mm to (205.8, 189.4)
- moved SW11 127.4 mm to (171.5, 193.8)
- moved SW1 123.1 mm to (205.8, 180.8)
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Connections:
- Q1 pad 2: /Display_interface/AN0 -> /Display_interface/AN3
- Q2 pad 2: /Display_interface/AN1 -> /Display_interface/AN0
- Q3 pad 2: /Display_interface/AN2 -> /Display_interface/AN1
- Q4 pad 2: /Display_interface/AN3 -> /Display_interface/AN2
- R1 pad 1: Net-(U2-ADJ) -> Net-(D1-A)
- R1 pad 2: /Power_Supply/+3v3 -> /Power_Supply/+5V
- R10 pad 1: /Display_interface/SEG_D -> /Display_interface/SEG_B
- R10 pad 2: /Display_interface/SEG_D -> /Display_interface/SEG_B
- R12 pad 1: /Coin_Buttons/BTNL -> /Display_interface/AN3
- R12 pad 2: GND -> /Display_interface/AN3
- R13 pad 1: /Coin_Buttons/BTNR -> /Display_interface/AN0
- R13 pad 2: GND -> /Display_interface/AN0
- R14 pad 1: /Coin_Buttons/BTND -> /Display_interface/AN1
- R14 pad 2: GND -> /Display_interface/AN1
- R15 pad 1: /Coin_Buttons/BTNU -> /Display_interface/AN2
- R15 pad 2: GND -> /Display_interface/AN2
- R16 pad 1: /Coin_Buttons/BTNC -> GND
- R16 pad 2: GND -> /FPGA_IO/LED1
- R17 pad 2: /FPGA_IO/LED0 -> /FPGA_IO/LED2
- R18 pad 2: /FPGA_IO/LED1 -> /FPGA_IO/LED0
- R19 pad 1: GND -> Net-(D2-A)
- R19 pad 2: /FPGA_IO/LED2 -> +5V
- R2 pad 2: GND -> /Power_Supply/+3v3
- R20 pad 1: /Display_interface/SEG_C -> /Coin_Buttons/BTNL
- R20 pad 2: /Display_interface/SEG_C -> /FPGA_IO/+3v3
- R21 pad 1: /Display_interface/SEG_D -> /Coin_Buttons/BTNR
- R21 pad 2: /Display_interface/SEG_D -> GND
- R22 pad 1: /Display_interface/SEG_D -> /Coin_Buttons/BTNC
- R22 pad 2: /Display_interface/SEG_D -> /FPGA_IO/+3v3
- R23 pad 1: /Display_interface/SEG_F -> /Coin_Buttons/BTNU
- R23 pad 2: /Display_interface/SEG_F -> /FPGA_IO/+3v3
- R24 pad 1: /Display_interface/SEG_A -> /Coin_Buttons/BTND
- R24 pad 2: /Display_interface/SEG_A -> GND
- R25 pad 1: /Display_interface/SEG_D -> Net-(U6-ADJ)
- R25 pad 2: /Display_interface/SEG_D -> /FPGA_IO/+3v3
- R26 pad 1: /Display_interface/SEG_B -> Net-(U6-ADJ)
- R26 pad 2: /Display_interface/SEG_B -> GND
- R27 pad 1: /Display_interface/SEG_D -> /Display_interface/SEG_C
- R27 pad 2: /Display_interface/SEG_D -> /Display_interface/SEG_C
- R28 pad 1: /Coin_Buttons/BTNL -> /Display_interface/SEG_D
- R28 pad 2: /FPGA_IO/+3v3 -> /Display_interface/SEG_D
- R29 pad 1: /Coin_Buttons/BTNR -> /Display_interface/SEG_D
- R29 pad 2: GND -> /Display_interface/SEG_D
- R3 pad 1: Net-(D1-A) -> Net-(U2-ADJ)
- R3 pad 2: /Power_Supply/+5V -> GND
- R30 pad 1: /Coin_Buttons/BTNC -> /Display_interface/SEG_F
- R30 pad 2: /FPGA_IO/+3v3 -> /Display_interface/SEG_F
- R31 pad 1: /Coin_Buttons/BTNU -> /Display_interface/SEG_A
- R31 pad 2: /FPGA_IO/+3v3 -> /Display_interface/SEG_A
- R32 pad 1: /Coin_Buttons/BTND -> /Display_interface/SEG_D
- R32 pad 2: GND -> /Display_interface/SEG_D
- R33 pad 1: Net-(D2-A) -> /Display_interface/SEG_B
- R33 pad 2: +5V -> /Display_interface/SEG_B
- R34 pad 1: Net-(U7-ADJ) -> /Display_interface/SEG_D
- R34 pad 2: /FPGA_IO/+3v3 -> /Display_interface/SEG_D
- R35 pad 1: Net-(U7-ADJ) -> /Display_interface/AN3
- R35 pad 2: GND -> /Display_interface/AN3
- R4 pad 1: /Display_interface/SEG_A -> /Display_interface/SEG_C
- R4 pad 2: /Display_interface/SEG_A -> /Display_interface/SEG_C
- R5 pad 1: /Display_interface/SEG_B -> /Display_interface/SEG_D
- R5 pad 2: /Display_interface/SEG_B -> /Display_interface/SEG_D
- R6 pad 1: /Display_interface/SEG_C -> /Display_interface/SEG_D
- R6 pad 2: /Display_interface/SEG_C -> /Display_interface/SEG_D
- R7 pad 1: /Display_interface/SEG_D -> /Display_interface/SEG_F
- R7 pad 2: /Display_interface/SEG_D -> /Display_interface/SEG_F
- R8 pad 1: /Display_interface/SEG_D -> /Display_interface/SEG_A
- R8 pad 2: /Display_interface/SEG_D -> /Display_interface/SEG_A
- R9 pad 1: /Display_interface/SEG_F -> /Display_interface/SEG_D
- R9 pad 2: /Display_interface/SEG_F -> /Display_interface/SEG_D
- SW1 pad 1: +3.3V -> /Power_Supply/Vin
- SW1 pad 2: /Coin_Buttons/BTNR -> /Power_Supply/+3v3
- SW10 pad 2: /Coin_Buttons/BTNC -> /Coin_Buttons/BTNL
- SW11 pad 2: /Coin_Buttons/BTNU -> /Coin_Buttons/BTNC
- SW12 pad 1: /FPGA_IO/Vin -> +3.3V
- SW12 pad 2: /FPGA_IO/+3v3 -> /Coin_Buttons/BTNU
- SW2 pad 2: /Coin_Buttons/BTND -> /Coin_Buttons/BTNR
- SW3 pad 1: /Power_Supply/Vin -> +3.3V
- SW3 pad 2: /Power_Supply/+3v3 -> /Coin_Buttons/BTND
- SW4 pad 2: /Coin_Buttons/BTNC -> /Coin_Buttons/BTNL
- SW5 pad 2: /Coin_Buttons/BTNU -> /Coin_Buttons/BTNC
- SW6 pad 2: /Coin_Buttons/BTNL -> /Coin_Buttons/BTNU
- SW7 pad 1: +3.3V -> /FPGA_IO/Vin
- SW7 pad 2: /Coin_Buttons/BTNR -> /FPGA_IO/+3v3
- SW8 pad 2: /Coin_Buttons/BTND -> /Coin_Buttons/BTNR
- SW9 pad 2: /Coin_Buttons/BTNL -> /Coin_Buttons/BTND
- U3 pad 12: Net-(Q1-C) -> Net-(Q2-C)
- U3 pad 6: Net-(Q4-C) -> Net-(Q1-C)
- U3 pad 8: Net-(Q3-C) -> Net-(Q4-C)
- U3 pad 9: Net-(Q2-C) -> Net-(Q3-C)
- U4 pad B1: unconnected-(U4A-VCCO_15-PadB1) -> /FPGA_IO/+3v3
- U4 pad N4: unconnected-(U4A-VCCO_15-PadN4) -> /FPGA_IO/+3v3
- U4 pad P12: unconnected-(U4A-VCCO_15-PadP12) -> /FPGA_IO/+3v3
- U4 pad R1: unconnected-(U4A-VCCO_15-PadR1) -> /FPGA_IO/+3v3
- U5 pad 1: /Display_interface/SEG_D -> /FPGA_IO/Vin
- U5 pad 2: /Display_interface/SEG_D -> GND
- U5 pad 3: /Display_interface/SEG_D -> +5V
- U6 pad 1: /FPGA_IO/Vin -> Net-(U6-ADJ)
- U6 pad 2: GND -> /FPGA_IO/+3v3
- U6 pad 3: +5V -> Net-(U6-VI)
- U7 pad 1: Net-(U7-ADJ) -> /Display_interface/SEG_D
- U7 pad 2: /FPGA_IO/+3v3 -> /Display_interface/SEG_D
- U7 pad 3: Net-(U7-VI) -> /Display_interface/SEG_D
Routing:
- net GND: track 0.00 -> 276.5 mm, vias 0 -> 1
- net /Coin_Buttons/BTNR: track 0.00 -> 269.2 mm, vias 0 -> 1
- net /Display_interface/SEG_D: track 0.00 -> 266.0 mm
- net /Coin_Buttons/BTND: track 0.00 -> 240.0 mm, vias 0 -> 2
- net +3.3V: track 0.00 -> 235.0 mm, vias 0 -> 5
- net /Coin_Buttons/BTNC: track 0.00 -> 195.0 mm, vias 0 -> 2
- net /Display_interface/SEG_F: track 0.00 -> 190.9 mm, vias 0 -> 2
- net /FPGA_IO/+3v3: track 0.00 -> 187.3 mm, vias 0 -> 3
- net /Display_interface/AN3: track 0.00 -> 182.2 mm, vias 0 -> 5
- net /Display_interface/SEG_C: track 0.00 -> 177.4 mm, vias 0 -> 2
- net /Coin_Buttons/BTNU: track 0.00 -> 173.5 mm, vias 0 -> 2
- net /Display_interface/AN1: track 0.00 -> 152.6 mm, vias 0 -> 5
- net /Coin_Buttons/BTNL: track 0.00 -> 149.1 mm, vias 0 -> 1
- net +5V: track 0.00 -> 148.5 mm, vias 0 -> 2
- net /Display_interface/SEG_B: track 0.00 -> 135.6 mm, vias 0 -> 2
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Other:
- board outline added: 113 x 123.5 mm
